Commit message: update urdf

File: urdf/wow_body_little.urdf (robot description, URDF)
Before this commit: robot up_body, 18 links, 17 joints
Links:
- link base: geometry collision mesh filename=package://wow_description/robot/wow_little/meshes/base.STL; visual mesh filename=package://wow_description/robot/wow_little/meshes/base.STL
- link left_1_link: geometry collision mesh filename=package://wow_description/robot/wow_little/meshes/left_1_li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; visual mesh filename=package://wow_description/robot/wow_little/meshes/left_1_li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
- link left_2_link: geometry collision mesh filename=package://wow_description/robot/wow_little/meshes/left_2_li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; visual mesh filename=package://wow_description/robot/wow_little/meshes/left_2_li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
- link left_3_link: geometry collision mesh filename=package://wow_description/robot/wow_little/meshes/left_3_li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; visual mesh filename=package://wow_description/robot/wow_little/meshes/left_3_li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
- link left_4_link: geometry collision mesh filename=package://wow_description/robot/wow_little/meshes/left_4_li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; visual mesh filename=package://wow_description/robot/wow_little/meshes/left_4_li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
- link left_5_link: geometry collision mesh filename=package://wow_description/robot/wow_little/meshes/left_5_li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; visual mesh filename=package://wow_description/robot/wow_little/meshes/left_5_li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
- link left_6_link: geometry collision mesh filename=package://wow_description/robot/wow_little/meshes/left_6_li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; visual mesh filename=package://wow_description/robot/wow_little/meshes/left_6_li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
- link left_7_link: geometry collision mesh filename=package://wow_description/robot/wow_little/meshes/left_7_li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; visual mesh filename=package://wow_description/robot/wow_little/meshes/left_7_li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
- link left_8_link: geometry collision mesh filename=package://wow_description/robot/wow_little/meshes/left_8_li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; visual mesh filename=package://wow_description/robot/wow_little/meshes/left_8_li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
- link right_1_link: geometry collision mesh filename=package://wow_description/robot/wow_little/meshes/right_1_l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; visual mesh filename=package://wow_description/robot/wow_little/meshes/right_1_l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
- link right_2_link: geometry collision mesh filename=package://wow_description/robot/wow_little/meshes/right_2_l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; visual mesh filename=package://wow_description/robot/wow_little/meshes/right_2_l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
- link right_3_link: geometry collision mesh filename=package://wow_description/robot/wow_little/meshes/right_3_l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; visual mesh filename=package://wow_description/robot/wow_little/meshes/right_3_l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
- link right_4_link: geometry collision mesh filename=package://wow_description/robot/wow_little/meshes/right_4_l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; visual mesh filename=package://wow_description/robot/wow_little/meshes/right_4_l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
- link right_5_link: geometry collision mesh filename=package://wow_description/robot/wow_little/meshes/right_5_l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; visual mesh filename=package://wow_description/robot/wow_little/meshes/right_5_l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
- link right_6_link: geometry collision mesh filename=package://wow_description/robot/wow_little/meshes/right_6_l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; visual mesh filename=package://wow_description/robot/wow_little/meshes/right_6_l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
- link right_7_link: geometry collision mesh filename=package://wow_description/robot/wow_little/meshes/right_7_l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; visual mesh filename=package://wow_description/robot/wow_little/meshes/right_7_l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
- link right_8_link: geometry collision mesh filename=package://wow_description/robot/wow_little/meshes/right_8_l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; visual mesh filename=package://wow_description/robot/wow_little/meshes/right_8_l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
